File: nanoExpander_v12/nanoExpander_v12.kicad_pcb (KiCad board)
At the start: 2 copper layers, 60 x 71 mm, 37 parts, among them J00 Conn_01x04, J01 Conn_01x04, J02 Conn_01x04, J03 Conn_01x04, J04 Conn_01x04, J05 Conn_01x04, J06 Conn_01x04, J07 Conn_01x04, J08 Conn_01x04, J09 Conn_01x04, J10 Conn_01x04, J11 Conn_01x04, J12 Conn_01x02, J13 Conn_01x03, Q00 BSS138, SW00 ON/OFF, U00 ARDUINO_NANO_33_IOT, U01 MCP73831-2, U03 MIC5216

Commit message: Add files via upload
Parts:
- added J14: Conn_01x03, Connector_PinSocket_2.54mm:PinSocket_1x03_P2.54mm_Vertical, F.Cu at (83.0, 140.7)
- moved JP00 2.90 mm to (86.1, 135.1)
Connections:
- RN00 pad 1: D11 -> D13
- RN00 pad 3: D13 -> D11
Routing:
- net D13: track 66.5 -> 52.9 mm, vias 2 -> 0
- net D11: track 59.6 -> 57.4 mm, vias 2 -> 0
- net TX: track 53.9 -> 56.0 mm
- net RX: track 55.3 -> 57.2 mm
- net Net-(JP00-Pad2): track 34.5 -> 35.5 mm
