File: nanoExpander_v12/nanoExpander_v12.sch (KiCad schematic (older format))
At the start: 34 parts, among them J00 Conn_01x04, J01 Conn_01x04, J02 Conn_01x04, J03 Conn_01x04, J04 Conn_01x04, J05 Conn_01x04, J06 Conn_01x04, J07 Conn_01x04, J08 Conn_01x04, J09 Conn_01x04, J10 Conn_01x04, J11 Conn_01x04, J12 Conn_01x02, J13 Conn_01x03, Q00 BSS138, SW00 ON/OFF, U00 ARDUINO_NANO_33_IOT, U01 MCP73831-2, U03 MIC5216

Commit message: Add files via upload
Parts:
- added J14: Conn_01x03, Connector_PinSocket_2.54mm:PinSocket_1x03_P2.54mm_Vertical, symbol Connector_Generic:Conn_01x03
Connections:
- net D11: now also RN00.3 (R3.1); no longer RN00.1 (R1.1)
- net D13: now also RN00.1 (R1.1); no longer RN00.3 (R3.1)
- net GND: now also J14.3 (Pin_3)
- net VUSB: now also J14.1 (Pin_1)
- net at J13.2 (Pin_2), Q00.3 (D), R02.1: now also J14.2 (Pin_2)
Changed lines of the file:
@@
 Wire Wire Line
 	9300 2050 9200 2050
-Text GLabel 8100 2050 0    50   Input ~ 0
+Text GLabel 8100 1850 0    50   Input ~ 0
 D13
 Text GLabel 8100 1950 0    50   Input ~ 0
 D12
-Text GLabel 8100 1850 0    50   Input ~ 0
+Text GLabel 8100 2050 0    50   Input ~ 0
 D11
 Wire Wire Line
@@
 $EndComp
 Wire Wire Line
-	7800 5800 7550 5800
+	7800 5800 7700 5800
 Connection ~ 7550 5800
 Wire Wire Line
 	7400 5450 7550 5450
-Wire Wire Line
-	7800 5450 7800 5700
 Wire Wire Line
 	7550 5500 7550 5450
@@
 Text GLabel 6600 5450 0    50   Input ~ 0
 VUSB
+$Comp
+L Connector_Generic:Conn_01x03 J14
+U 1 1 5F19208D
+P 8600 5800
+F 0 "J14" H 8680 5842 50  0000 L CNN
+F 1 "Conn_01x03" H 8680 5751 50  0000 L CNN
+F 2 "Connector_PinSocket_2.54mm:PinSocket_1x03_P2.54mm_Vertical" H 8600 5800 50  0001 C CNN
+F 3 "~" H 8600 5800 50  0001 C CNN
+	1    8600 5800
+	1    0    0    -1
+$EndComp
+Wire Wire Line
+	7800 5450 8400 5450
+Wire Wire Line
+	8400 5450 8400 5700
+Connection ~ 7800 5450
+Wire Wire Line
+	7800 5450 7800 5700
+Wire Wire Line
+	7700 5800 7700 5550
+Wire Wire Line
+	7700 5550 8300 5550
+Wire Wire Line
+	8300 5550 8300 5800
+Wire Wire Line
+	8300 5800 8400 5800
+Connection ~ 7700 5800
+Wire Wire Line
+	7700 5800 7550 5800
+$Comp
+L power:GND #PWR?
+U 1 1 5F1A90B1
+P 8400 5900
+F 0 "#PWR?" H 8400 5650 50  0001 C CNN
+F 1 "GND" H 8405 5727 50  0000 C CNN
+F 2 "" H 8400 5900 50  0001 C CNN
+F 3 "" H 8400 5900 50  0001 C CNN
+	1    8400 5900
+	1    0    0    -1
+$EndComp
 $EndSCHEMATC
